File: pcb/diagnostic-port-dongle.kicad_sch (KiCad schematic)
At the start: 9 parts, among them J1 ODU Diagnostic Port, J2 Inverter Tester, J3 5V-3.3V Level Shifter, J4 XIAO ESP32S3, J5 ODU 5V power jumper

Commit message: added disclaimer
Parts:
- J1, J2: footprint midea:JST_XH_B4B-XH-A_1x04_P2.50mm_Vertical -> diagnostic-port-dongle:JST_XH_B4B-XH-A_1x04_P2.50mm_Vertical
- J3: footprint midea:Module_LevelShifter_4ch_2x06_P2.54mm_RM10.16 -> diagnostic-port-dongle:Module_LevelShifter_4ch_2x06_P2.54mm_RM10.16
- J4: footprint midea:Module_Seeed_XIAO_2x07_P2.54mm_RM15.24 -> diagnostic-port-dongle:Module_Seeed_XIAO_2x07_P2.54mm_RM15.24
Other:
- title: midea-telemetry ODU diagnostic-port adapter -> ODU diagnostic-port dongle
Changed lines of the file:
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@@
 	(paper "A4")
 	(title_block
-		(title "midea-telemetry ODU diagnostic-port adapter")
+		(title "ODU diagnostic-port dongle")
 		(rev "4")
-		(comment 1 "github.com/fmck3516/midea-telemetry")
+		(comment 1 "github.com/fmck3516/midea-telemetry-esphome")
 	)
 	(symbol
@@
 		(property "Reference" "J1" (at 44.45 41.910000000000004 0)  (effects (font (size 1.27 1.27))))
 		(property "Value" "ODU Diagnostic Port" (at 44.45 39.370000000000005 0)  (effects (font (size 1.27 1.27))))
-		(property "Footprint" "midea:JST_XH_B4B-XH-A_1x04_P2.50mm_Vertical" (at 46.99 53.34 0) (hide yes) (effects (font (size 1.27 1.27))))
+		(property "Footprint" "diagnostic-port-dongle:JST_XH_B4B-XH-A_1x04_P2.50mm_Vertical" (at 46.99 53.34 0) (hide yes) (effects (font (size 1.27 1.27))))
 		(property "Datasheet" "" (at 46.99 53.34 0) (hide yes) (effects (font (size 1.27 1.27))))
 		(property "Description" "" (at 46.99 53.34 0) (hide yes) (effects (font (size 1.27 1.27))))
@@
 		(pin "3")
 		(pin "4")
-		(instances (project "midea-telemetry-adapter" (path "/4cd5a3a6-441a-4d49-b89e-ac57047910ed" (reference "J1") (unit 1))))
+		(instances (project "diagnostic-port-dongle" (path "/4cd5a3a6-441a-4d49-b89e-ac57047910ed" (reference "J1") (unit 1))))
 	)
 	(wire (pts (xy 52.07 48.260000000000005) (xy 63.5 48.260000000000005)) (stroke (width 0) (type default)))
@@
 		(property "Reference" "J2" (at 44.45 69.85 0)  (effects (font (size 1.27 1.27))))
 		(property "Value" "Inverter Tester" (at 44.45 67.31 0)  (effects (font (size 1.27 1.27))))
-		(property "Footprint" "midea:JST_XH_B4B-XH-A_1x04_P2.50mm_Vertical" (at 46.99 81.28 0) (hide yes) (effects (font (size 1.27 1.27))))
+		(property "Footprint" "diagnostic-port-dongle:JST_XH_B4B-XH-A_1x04_P2.50mm_Vertical" (at 46.99 81.28 0) (hide yes) (effects (font (size 1.27 1.27))))
 		(property "Datasheet" "" (at 46.99 81.28 0) (hide yes) (effects (font (size 1.27 1.27))))
 		(property "Description" "" (at 46.99 81.28 0) (hide yes) (effects (font (size 1.27 1.27))))
@@
 		(pin "3")
 		(pin "4")
-		(instances (project "midea-telemetry-adapter" (path "/4cd5a3a6-441a-4d49-b89e-ac57047910ed" (reference "J2") (unit 1))))
+		(instances (project "diagnostic-port-dongle" (path "/4cd5a3a6-441a-4d49-b89e-ac57047910ed" (reference "J2") (unit 1))))
 	)
 	(wire (pts (xy 52.07 76.2) (xy 63.5 76.2)) (stroke (width 0) (type default)))
@@
 		(property "Reference" "J3" (at 102.86999999999999 48.260000000000005 0)  (effects (font (size 1.27 1.27))))
 		(property "Value" "5V-3.3V Level Shifter" (at 102.86999999999999 45.72 0)  (effects (font (size 1.27 1.27))))
-		(property "Footprint" "midea:Module_LevelShifter_4ch_2x06_P2.54mm_RM10.16" (at 101.6 60.96 0) (hide yes) (effects (font (size 1.27 1.27))))
+		(property "Footprint" "diagnostic-port-dongle:Module_LevelShifter_4ch_2x06_P2.54mm_RM10.16" (at 101.6 60.96 0) (hide yes) (effects (font (size 1.27 1.27))))
 		(property "Datasheet" "" (at 101.6 60.96 0) (hide yes) (effects (font (size 1.27 1.27))))
 		(property "Description" "" (at 101.6 60.96 0) (hide yes) (effects (font (size 1.27 1.27))))
@@
 		(pin "11")
 		(pin "12")
-		(instances (project "midea-telemetry-adapter" (path "/4cd5a3a6-441a-4d49-b89e-ac57047910ed" (reference "J3") (unit 1))))
+		(instances (project "diagnostic-port-dongle" (path "/4cd5a3a6-441a-4d49-b89e-ac57047910ed" (reference "J3") (unit 1))))
 	)
 	(text "HV1" (exclude_from_sim no) (at 95.25 56.38 0) (effects (font (size 1.0 1.0)) (justify right)))
@@
 		(property "Reference" "J4" (at 165.10000000000002 48.26 0)  (effects (font (size 1.27 1.27))))
 		(property "Value" "XIAO ESP32S3" (at 165.10000000000002 45.72 0)  (effects (font (size 1.27 1.27))))
-		(property "Footprint" "midea:Module_Seeed_XIAO_2x07_P2.54mm_RM15.24" (at 163.83 63.5 0) (hide yes) (effects (font (size 1.27 1.27))))
+		(property "Footprint" "diagnostic-port-dongle:Module_Seeed_XIAO_2x07_P2.54mm_RM15.24" (at 163.83 63.5 0) (hide yes) (effects (font (size 1.27 1.27))))
 		(property "Datasheet" "" (at 163.83 63.5 0) (hide yes) (effects (font (size 1.27 1.27))))
 		(property "Description" "" (at 163.83 63.5 0) (hide yes) (effects (font (size 1.27 1.27))))
@@
 		(pin "13")
 		(pin "14")
-		(instances (project "midea-telemetry-adapter" (path "/4cd5a3a6-441a-4d49-b89e-ac57047910ed" (reference "J4") (unit 1))))
+		(instances (project "diagnostic-port-dongle" (path "/4cd5a3a6-441a-4d49-b89e-ac57047910ed" (reference "J4") (unit 1))))
 	)
 	(text "D0" (exclude_from_sim no) (at 157.48 56.38 0) (effects (font (size 1.0 1.0)) (justify right)))
@@
 		(pin "1")
 		(pin "2")
-		(instances (project "midea-telemetry-adapter" (path "/4cd5a3a6-441a-4d49-b89e-ac57047910ed" (reference "J5") (unit 1))))
+		(instances (project "diagnostic-port-dongle" (path "/4cd5a3a6-441a-4d49-b89e-ac57047910ed" (reference "J5") (unit 1))))
 	)
 	(wire (pts (xy 96.52 88.9) (xy 83.82 88.9)) (stroke (width 0) (type default)))
@@
 		(property "Datasheet" "" (at 144.78 152.4 0) (hide yes) (effects (font (size 1.27 1.27))))
 		(property "Description" "" (at 144.78 152.4 0) (hide yes) (effects (font (size 1.27 1.27))))
-		(instances (project "midea-telemetry-adapter" (path "/4cd5a3a6-441a-4d49-b89e-ac57047910ed" (reference "H1") (unit 1))))
+		(instances (project "diagnostic-port-dongle" (path "/4cd5a3a6-441a-4d49-b89e-ac57047910ed" (reference "H1") (unit 1))))
 	)
 	(symbol
@@
 		(property "Datasheet" "" (at 153.67 152.4 0) (hide yes) (effects (font (size 1.27 1.27))))
 		(property "Description" "" (at 153.67 152.4 0) (hide yes) (effects (font (size 1.27 1.27))))
-		(instances (project "midea-telemetry-adapter" (path "/4cd5a3a6-441a-4d49-b89e-ac57047910ed" (reference "H2") (unit 1))))
+		(instances (project "diagnostic-port-dongle" (path "/4cd5a3a6-441a-4d49-b89e-ac57047910ed" (reference "H2") (unit 1))))
 	)
 	(symbol
@@
 		(property "Datasheet" "" (at 162.56 152.4 0) (hide yes) (effects (font (size 1.27 1.27))))
 		(property "Description" "" (at 162.56 152.4 0) (hide yes) (effects (font (size 1.27 1.27))))
-		(instances (project "midea-telemetry-adapter" (path "/4cd5a3a6-441a-4d49-b89e-ac57047910ed" (reference "H3") (unit 1))))
+		(instances (project "diagnostic-port-dongle" (path "/4cd5a3a6-441a-4d49-b89e-ac57047910ed" (reference "H3") (unit 1))))
 	)
 	(symbol
@@
 		(property "Datasheet" "" (at 171.45 152.4 0) (hide yes) (effects (font (size 1.27 1.27))))
 		(property "Description" "" (at 171.45 152.4 0) (hide yes) (effects (font (size 1.27 1.27))))
-		(instances (project "midea-telemetry-adapter" (path "/4cd5a3a6-441a-4d49-b89e-ac57047910ed" (reference "H4") (unit 1))))
+		(instances (project "diagnostic-port-dongle" (path "/4cd5a3a6-441a-4d49-b89e-ac57047910ed" (reference "H4") (unit 1))))
 	)
 	(text "M2 mounting holes" (exclude_from_sim no) (at 144.78 144.78 0) (effects (font (size 1.27 1.27)) (justify left)))
