File: pcb/diagnostic-port-dongle.kicad_pcb (KiCad board)
At the start: 2 copper layers, 57 x 30 mm, 9 parts, among them J1 ODU Diagnostic Port, J2 Inverter Tester, J3 5V-3.3V Level Shifter, J4 XIAO ESP32S3, J5 ODU 5V power jumper

Commit message: added disclaimer
Parts:
- J1, J2: footprint midea:JST_XH_B4B-XH-A_1x04_P2.50mm_Vertical -> diagnostic-port-dongle:JST_XH_B4B-XH-A_1x04_P2.50mm_Vertical
- J3: footprint midea:Module_LevelShifter_4ch_2x06_P2.54mm_RM10.16 -> diagnostic-port-dongle:Module_LevelShifter_4ch_2x06_P2.54mm_RM10.16
- J4: footprint midea:Module_Seeed_XIAO_2x07_P2.54mm_RM15.24 -> diagnostic-port-dongle:Module_Seeed_XIAO_2x07_P2.54mm_RM15.24
Other:
- board text added: "ODU diagnostic-port dongle"
- board text added: "github.com/fmck3516/midea-telemetry-esphome"
- board text removed: "ODU diagnostic-port adapter - rev 4"
- board text removed: "github.com/fmck3516/midea-telemetry"
- board text removed: "midea-telemetry"
Changed lines of the file:
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@@
 		(embedded_fonts no)
 	)
-	(footprint "midea:Module_Seeed_XIAO_2x07_P2.54mm_RM15.24"
+	(footprint "diagnostic-port-dongle:Module_Seeed_XIAO_2x07_P2.54mm_RM15.24"
 		(layer "F.Cu")
 		(at 47.9 15)
@@
 		(embedded_fonts no)
 	)
-	(footprint "midea:JST_XH_B4B-XH-A_1x04_P2.50mm_Vertical"
+	(footprint "diagnostic-port-dongle:JST_XH_B4B-XH-A_1x04_P2.50mm_Vertical"
 		(layer "F.Cu")
 		(at 16 18.75 90)
@@
 		)
 	)
-	(footprint "midea:Module_LevelShifter_4ch_2x06_P2.54mm_RM10.16"
+	(footprint "diagnostic-port-dongle:Module_LevelShifter_4ch_2x06_P2.54mm_RM10.16"
 		(layer "F.Cu")
 		(at 29.58 15 90)
@@
 		(embedded_fonts no)
 	)
-	(footprint "midea:JST_XH_B4B-XH-A_1x04_P2.50mm_Vertical"
+	(footprint "diagnostic-port-dongle:JST_XH_B4B-XH-A_1x04_P2.50mm_Vertical"
 		(layer "F.Cu")
 		(at 4.5 18.75 90)
@@
 		)
 	)
-	(gr_text "ODU diagnostic-port adapter  -  rev 4"
-		(at 28.5 28.4 0)
-		(layer "F.SilkS")
-		(effects
-			(font
-				(size 0.85 0.85)
-				(thickness 0.14)
-			)
-		)
-	)
-	(gr_text "github.com/fmck3516/midea-telemetry"
+	(gr_text "github.com/fmck3516/midea-telemetry-esphome"
 		(at 28.5 2.5 0)
 		(layer "F.SilkS")
@@
 		)
 	)
-	(gr_text "midea-telemetry"
-		(at 28.5 26.4 0)
+	(gr_text "ODU diagnostic-port dongle"
+		(at 28.5 27.6 0)
 		(layer "F.SilkS")
 		(effects
 			(font
-				(size 1.4 1.4)
-				(thickness 0.28)
+				(size 1.0 1.0)
+				(thickness 0.2)
 				(bold yes)
 			)

Commit message: more work on enclosure
Other:
- board text removed: "github.com/fmck3516/midea-telemetry-esphome"
Changed lines of the file:
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@@
-		)
-	)
-	(gr_text "github.com/fmck3516/midea-telemetry-esphome"
-		(at 28.5 2.5 0)
-		(layer "F.SilkS")
-		(effects
-			(font
-				(size 0.95 0.95)
-				(thickness 0.14)
-			)
 		)
 	)
