File: pcb/telemetry-module.kicad_sch (KiCad schematic)
At the start: 9 parts, among them J1 ODU Diagnostic Port, J2 Inverter Tester, J3 5V-3.3V Level Shifter, J4 XIAO ESP32S3, J5 ODU 5V power jumper

Commit message: more work on PCB
Parts:
- removed J2: Inverter Tester, diagnostic-port-dongle:JST_XH_B4B-XH-A_1x04_P2.50mm_Vertical, symbol Connector_Generic:Conn_01x04
- J1: footprint diagnostic-port-dongle:JST_XH_B4B-XH-A_1x04_P2.50mm_Vertical -> telemetry-module:JST_XH_B4B-XH-A_1x04_P2.50mm_Vertical
- J3: footprint diagnostic-port-dongle:Module_LevelShifter_4ch_2x06_P2.54mm_RM10.16 -> telemetry-module:Module_LevelShifter_4ch_2x06_P2.54mm_RM10.16
- J4: footprint diagnostic-port-dongle:Module_Seeed_XIAO_2x07_P2.54mm_RM15.24 -> telemetry-module:Module_Seeed_XIAO_2x07_P2.54mm_RM15.24
Other:
- note added: "J1 taps the ODU diagnostic port; the ESP32 reads the CLK / DAT bus through the level shifter."
- note removed: "J1 and J2 are wired 1:1 in parallel. Plug the ODU diagnostic port into either one; the other can"
- note removed: "carry the Midea inverter tester so the ESP32 can sniff the traffic between tester and ODU."
- note removed: "pass-through, for sniffing"
Changed lines of the file:
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@@
 	(title_block
 		(title "ODU diagnostic-port dongle")
-		(rev "4")
+		(rev "5")
 		(comment 1 "github.com/fmck3516/midea-telemetry-esphome")
 	)
@@
 		(property "Reference" "J1" (at 44.45 41.910000000000004 0)  (effects (font (size 1.27 1.27))))
 		(property "Value" "ODU Diagnostic Port" (at 44.45 39.370000000000005 0)  (effects (font (size 1.27 1.27))))
-		(property "Footprint" "diagnostic-port-dongle:JST_XH_B4B-XH-A_1x04_P2.50mm_Vertical" (at 46.99 53.34 0) (hide yes) (effects (font (size 1.27 1.27))))
+		(property "Footprint" "telemetry-module:JST_XH_B4B-XH-A_1x04_P2.50mm_Vertical" (at 46.99 53.34 0) (hide yes) (effects (font (size 1.27 1.27))))
 		(property "Datasheet" "" (at 46.99 53.34 0) (hide yes) (effects (font (size 1.27 1.27))))
 		(property "Description" "" (at 46.99 53.34 0) (hide yes) (effects (font (size 1.27 1.27))))
@@
 		(pin "3")
 		(pin "4")
-		(instances (project "diagnostic-port-dongle" (path "/4cd5a3a6-441a-4d49-b89e-ac57047910ed" (reference "J1") (unit 1))))
+		(instances (project "telemetry-module" (path "/4cd5a3a6-441a-4d49-b89e-ac57047910ed" (reference "J1") (unit 1))))
 	)
 	(wire (pts (xy 52.07 48.260000000000005) (xy 63.5 48.260000000000005)) (stroke (width 0) (type default)))
@@
 	(text "to the outdoor unit" (exclude_from_sim no) (at 44.45 63.5 0) (effects (font (size 1.0 1.0)) (justify left)))
 	(symbol
-		(lib_id "Connector_Generic:Conn_01x04")
-		(at 46.99 81.28 180)
-		(unit 1)
-		(body_style 1)
-		(exclude_from_sim no)(in_bom yes)(on_board yes)(dnp no)
-		(property "Reference" "J2" (at 44.45 69.85 0)  (effects (font (size 1.27 1.27))))
-		(property "Value" "Inverter Tester" (at 44.45 67.31 0)  (effects (font (size 1.27 1.27))))
-		(property "Footprint" "diagnostic-port-dongle:JST_XH_B4B-XH-A_1x04_P2.50mm_Vertical" (at 46.99 81.28 0) (hide yes) (effects (font (size 1.27 1.27))))
-		(property "Datasheet" "" (at 46.99 81.28 0) (hide yes) (effects (font (size 1.27 1.27))))
-		(property "Description" "" (at 46.99 81.28 0) (hide yes) (effects (font (size 1.27 1.27))))
-		(pin "1")
-		(pin "2")
-		(pin "3")
-		(pin "4")
-		(instances (project "diagnostic-port-dongle" (path "/4cd5a3a6-441a-4d49-b89e-ac57047910ed" (reference "J2") (unit 1))))
-	)
-	(wire (pts (xy 52.07 76.2) (xy 63.5 76.2)) (stroke (width 0) (type default)))
-	(label "ODU_5V" (at 63.5 76.2 0) (effects (font (size 1.27 1.27)) (justify left bottom)))
-	(text "VCC" (exclude_from_sim no) (at 43.18 76.7 0) (effects (font (size 1.0 1.0)) (justify right)))
-	(wire (pts (xy 52.07 78.74) (xy 63.5 78.74)) (stroke (width 0) (type default)))
-	(label "GND" (at 63.5 78.74 0) (effects (font (size 1.27 1.27)) (justify left bottom)))
-	(text "GND" (exclude_from_sim no) (at 43.18 79.24 0) (effects (font (size 1.0 1.0)) (justify right)))
-	(wire (pts (xy 52.07 81.28) (xy 63.5 81.28)) (stroke (width 0) (type default)))
-	(label "CLK_5V" (at 63.5 81.28 0) (effects (font (size 1.27 1.27)) (justify left bottom)))
-	(text "CLK" (exclude_from_sim no) (at 43.18 81.78 0) (effects (font (size 1.0 1.0)) (justify right)))
-	(wire (pts (xy 52.07 83.82000000000001) (xy 63.5 83.82000000000001)) (stroke (width 0) (type default)))
-	(label "DAT_5V" (at 63.5 83.82000000000001 0) (effects (font (size 1.27 1.27)) (justify left bottom)))
-	(text "DAT" (exclude_from_sim no) (at 43.18 84.32000000000001 0) (effects (font (size 1.0 1.0)) (justify right)))
-	(text "pass-through, for sniffing" (exclude_from_sim no) (at 44.45 91.44 0) (effects (font (size 1.0 1.0)) (justify left)))
-	(symbol
 		(lib_id "Connector_Generic:Conn_02x06_Odd_Even")
 		(at 101.6 60.96 0)
@@
 		(property "Reference" "J3" (at 102.86999999999999 48.260000000000005 0)  (effects (font (size 1.27 1.27))))
 		(property "Value" "5V-3.3V Level Shifter" (at 102.86999999999999 45.72 0)  (effects (font (size 1.27 1.27))))
-		(property "Footprint" "diagnostic-port-dongle:Module_LevelShifter_4ch_2x06_P2.54mm_RM10.16" (at 101.6 60.96 0) (hide yes) (effects (font (size 1.27 1.27))))
+		(property "Footprint" "telemetry-module:Module_LevelShifter_4ch_2x06_P2.54mm_RM10.16" (at 101.6 60.96 0) (hide yes) (effects (font (size 1.27 1.27))))
 		(property "Datasheet" "" (at 101.6 60.96 0) (hide yes) (effects (font (size 1.27 1.27))))
 		(property "Description" "" (at 101.6 60.96 0) (hide yes) (effects (font (size 1.27 1.27))))
@@
 		(pin "11")
 		(pin "12")
-		(instances (project "diagnostic-port-dongle" (path "/4cd5a3a6-441a-4d49-b89e-ac57047910ed" (reference "J3") (unit 1))))
+		(instances (project "telemetry-module" (path "/4cd5a3a6-441a-4d49-b89e-ac57047910ed" (reference "J3") (unit 1))))
 	)
 	(text "HV1" (exclude_from_sim no) (at 95.25 56.38 0) (effects (font (size 1.0 1.0)) (justify right)))
@@
 		(property "Reference" "J4" (at 165.10000000000002 48.26 0)  (effects (font (size 1.27 1.27))))
 		(property "Value" "XIAO ESP32S3" (at 165.10000000000002 45.72 0)  (effects (font (size 1.27 1.27))))
-		(property "Footprint" "diagnostic-port-dongle:Module_Seeed_XIAO_2x07_P2.54mm_RM15.24" (at 163.83 63.5 0) (hide yes) (effects (font (size 1.27 1.27))))
+		(property "Footprint" "telemetry-module:Module_Seeed_XIAO_2x07_P2.54mm_RM15.24" (at 163.83 63.5 0) (hide yes) (effects (font (size 1.27 1.27))))
 		(property "Datasheet" "" (at 163.83 63.5 0) (hide yes) (effects (font (size 1.27 1.27))))
 		(property "Description" "" (at 163.83 63.5 0) (hide yes) (effects (font (size 1.27 1.27))))
@@
 		(pin "13")
 		(pin "14")
-		(instances (project "diagnostic-port-dongle" (path "/4cd5a3a6-441a-4d49-b89e-ac57047910ed" (reference "J4") (unit 1))))
+		(instances (project "telemetry-module" (path "/4cd5a3a6-441a-4d49-b89e-ac57047910ed" (reference "J4") (unit 1))))
 	)
 	(text "D0" (exclude_from_sim no) (at 157.48 56.38 0) (effects (font (size 1.0 1.0)) (justify right)))
@@
 		(pin "1")
 		(pin "2")
-		(instances (project "diagnostic-port-dongle" (path "/4cd5a3a6-441a-4d49-b89e-ac57047910ed" (reference "J5") (unit 1))))
+		(instances (project "telemetry-module" (path "/4cd5a3a6-441a-4d49-b89e-ac57047910ed" (reference "J5") (unit 1))))
 	)
 	(wire (pts (xy 96.52 88.9) (xy 83.82 88.9)) (stroke (width 0) (type default)))
@@
 	(label "XIAO_5V" (at 83.82 91.44000000000001 0) (effects (font (size 1.27 1.27)) (justify right bottom)))
 	(text "fit the shunt to power the XIAO from the ODU" (exclude_from_sim no) (at 104.14 87.9 0) (effects (font (size 1.0 1.0)) (justify left)))
-	(text "J1 and J2 are wired 1:1 in parallel. Plug the ODU diagnostic port into either one; the other can" (exclude_from_sim no) (at 43.18 102.87 0) (effects (font (size 1.27 1.27)) (justify left)))
-	(text "carry the Midea inverter tester so the ESP32 can sniff the traffic between tester and ODU." (exclude_from_sim no) (at 43.18 107.95 0) (effects (font (size 1.27 1.27)) (justify left)))
+	(text "J1 taps the ODU diagnostic port; the ESP32 reads the CLK / DAT bus through the level shifter." (exclude_from_sim no) (at 43.18 102.87 0) (effects (font (size 1.27 1.27)) (justify left)))
 	(text "The 5V bus (CLK / DAT) is level-shifted to 3V3. The ODU supplies the 5V HV reference; the XIAO" (exclude_from_sim no) (at 43.18 113.03 0) (effects (font (size 1.27 1.27)) (justify left)))
 	(text "supplies the 3V3 LV reference." (exclude_from_sim no) (at 43.18 118.11 0) (effects (font (size 1.27 1.27)) (justify left)))
@@
 		(property "Datasheet" "" (at 144.78 152.4 0) (hide yes) (effects (font (size 1.27 1.27))))
 		(property "Description" "" (at 144.78 152.4 0) (hide yes) (effects (font (size 1.27 1.27))))
-		(instances (project "diagnostic-port-dongle" (path "/4cd5a3a6-441a-4d49-b89e-ac57047910ed" (reference "H1") (unit 1))))
+		(instances (project "telemetry-module" (path "/4cd5a3a6-441a-4d49-b89e-ac57047910ed" (reference "H1") (unit 1))))
 	)
 	(symbol
@@
 		(property "Datasheet" "" (at 153.67 152.4 0) (hide yes) (effects (font (size 1.27 1.27))))
 		(property "Description" "" (at 153.67 152.4 0) (hide yes) (effects (font (size 1.27 1.27))))
-		(instances (project "diagnostic-port-dongle" (path "/4cd5a3a6-441a-4d49-b89e-ac57047910ed" (reference "H2") (unit 1))))
+		(instances (project "telemetry-module" (path "/4cd5a3a6-441a-4d49-b89e-ac57047910ed" (reference "H2") (unit 1))))
 	)
 	(symbol
@@
 		(property "Datasheet" "" (at 162.56 152.4 0) (hide yes) (effects (font (size 1.27 1.27))))
 		(property "Description" "" (at 162.56 152.4 0) (hide yes) (effects (font (size 1.27 1.27))))
-		(instances (project "diagnostic-port-dongle" (path "/4cd5a3a6-441a-4d49-b89e-ac57047910ed" (reference "H3") (unit 1))))
+		(instances (project "telemetry-module" (path "/4cd5a3a6-441a-4d49-b89e-ac57047910ed" (reference "H3") (unit 1))))
 	)
 	(symbol
@@
 		(property "Datasheet" "" (at 171.45 152.4 0) (hide yes) (effects (font (size 1.27 1.27))))
 		(property "Description" "" (at 171.45 152.4 0) (hide yes) (effects (font (size 1.27 1.27))))
-		(instances (project "diagnostic-port-dongle" (path "/4cd5a3a6-441a-4d49-b89e-ac57047910ed" (reference "H4") (unit 1))))
+		(instances (project "telemetry-module" (path "/4cd5a3a6-441a-4d49-b89e-ac57047910ed" (reference "H4") (unit 1))))
 	)
 	(text "M2 mounting holes" (exclude_from_sim no) (at 144.78 144.78 0) (effects (font (size 1.27 1.27)) (justify left)))
