File: pcb/telemetry-module.kicad_pcb (KiCad board)
At the start: 2 copper layers, 41.5 x 22 mm, 8 parts, among them J1 ODU Diagnostic Port, J3 5V-3.3V Level Shifter, J4 XIAO ESP32S3, J5 ODU 5V power jumper

Commit message: Rename "diagnostic port" to "test port", Midea's name for it (issue #57)
Midea calls the outdoor unit's 4-pin service connector the test port:
it is labeled TEST on the control board. The repo called it the
diagnostic port, which matches neither the board nor the service
manuals, and the README said "diagnostic port" and "labeled TEST" in
the same sentence.

Test port now names the connector in README.md, UART-comparison.md
(prose and column header), FRAME-BYTES.md, the MideaTelemetry class
comment, the KiCad schematic (title block, J1 note, J1 value) and the
PCB (J1 value). "Diagnostic bus" wording is rephrased around the test
port too.

Left as is on purpose:
- the Medium article's title "Reverse Engineering Midea's ODU
  Diagnostic Port", where it is quoted, since that is its real title
  and its URL;
- Home Assistant's Diagnostic entity category;
- "the unit's own diagnostic display", which is the display, not the
  port.

J1's PCB value is on F.Fab, which is not part of the rev5 Gerber zip,
so the manufactured board is unchanged. pcb/schematic.png is
regenerated with kicad-cli 10.0.6 (PDF export without drawing sheet or
background) and trimmed to the original's width and margins. It now
also shows a GND power symbol that was already in the schematic source
but missing from the old render.

Checked: git grep -i diagnostic now finds only the three kept uses, and
the export left the KiCad sources untouched apart from the four
intended strings.

Co-Authored-By: Claude Opus 5 <noreply@anthropic.com>
Parts:
- J1: value ODU Diagnostic Port -> ODU Test Port
Changed lines of the file:
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@@
 			)
 		)
-		(property "Value" "ODU Diagnostic Port"
+		(property "Value" "ODU Test Port"
 			(at 3.75 4.6 0)
 			(layer "F.Fab")
